Commit message: 1走路1

File: resources/robots/bubble/urdf/bubble.urdf (robot description, URDF)
Before this commit: robot bubble, 9 links, 8 joints
Joints:
- joint left_knee_joint: axis 0.0 -1.0 0.0 -> 0.0 1.0 0.0
- joint left_wheel_joint: axis 0.0 -1.0 0.0 -> 0.0 1.0 0.0; limit (none) -> lower=-10000 upper=10000 effort=2.0 velocity=30.0; type continuous -> revolute
- joint right_knee_joint: limit lower=-0.436332 upper=0.488692 effort=2 velocity=100 -> lower=-0.488692 upper=0.436332 effort=2 velocity=100
- joint right_thigh_joint: axis 0.0 1.0 0.0 -> 0.0 -1.0 0.0; limit lower=-0.4 upper=0.7 effort=2 velocity=100 -> lower=-0.7 upper=0.4 effort=2 velocity=100
- joint right_wheel_joint: limit (none) -> lower=-10000 upper=10000 effort=2.0 velocity=30.0; type continuous -> revolute

Commit message: 平稳站立

File: resources/robots/bubble/urdf/bubble.urdf (robot description, URDF)
Before this commit: robot bubble, 9 links, 8 joints
Joints:
- joint left_wheel_joint: axis 0.0 1.0 0.0 -> 0.0 -1.0 0.0

Commit message: 小力矩能站立

File: resources/robots/bubble/urdf/bubble.urdf (robot description, URDF)
Before this commit: robot bubble, 9 links, 8 joints
Links:
- link base_link: mass 1.0 -> 0.7
- link left_thigh_link_1: mass 0.3 -> 0.21
- link right_thigh_link_1: mass 0.3 -> 0.21
Joints:
- joint left_knee_joint: limit lower=-0.436332 upper=0.488692 effort=2 velocity=100 -> lower=-0.436332 upper=0.488692 effort=0.5 velocity=100
- joint left_thigh_joint: limit lower=-0.4 upper=0.7 effort=2 velocity=100 -> lower=-0.4 upper=0.7 effort=0.5 velocity=100
- joint left_wheel_joint: limit lower=-10000 upper=10000 effort=2.0 velocity=30.0 -> lower=-10000 upper=10000 effort=0.5 velocity=30.0
- joint right_knee_joint: limit lower=-0.488692 upper=0.436332 effort=2 velocity=100 -> lower=-0.488692 upper=0.436332 effort=0.5 velocity=100
- joint right_thigh_joint: limit lower=-0.7 upper=0.4 effort=2 velocity=100 -> lower=-0.7 upper=0.4 effort=0.5 velocity=100
- joint right_wheel_joint: limit lower=-10000 upper=10000 effort=2.0 velocity=30.0 -> lower=-10000 upper=10000 effort=0.5 velocity=30.0

Commit message: 跟踪高度ok

File: resources/robots/bubble/urdf/bubble.urdf (robot description, URDF)
Before this commit: robot bubble, 9 links, 8 joints
Joints:
- joint left_thigh_joint: limit lower=-0.4 upper=0.7 effort=0.5 velocity=100 -> lower=-0.8 upper=1.2 effort=0.5 velocity=100
- joint right_thigh_joint: limit lower=-0.7 upper=0.4 effort=0.5 velocity=100 -> lower=-1.2 upper=0.8 effort=0.5 velocity=100
